Commit message: added lidar and joint state publishers to description
Signed-off-by: lkw303 <lkw303@gmail.com>

File: unodopo_description/urdf/unodopo.gazebo.xacro (robot description, xacro)
@@ -1,5 +1,5 @@
 <?xml version="1.0"?>
 <robot name="UnoDopo_sim" xmlns:xacro="http://www.ros.org/wiki/xacro">
-    <xacro:include filename="$(find urdf_tutorial)/urdf/uno_dopo_properties.urdf.xacro"/>
+    <xacro:include filename="$(find unodopo_description)/urdf/unodopo_properties.urdf.xacro"/>
     <!-- main wheel macro -->
     <xacro:macro name="main_wheels" params="suffix reflect">
@@ -17,5 +17,5 @@
     <xacro:main_wheels suffix="right" reflect="1.0"/>
     <xacro:main_wheels suffix="left" reflect="-1.0"/>
-    <gazebo reference="front_castor_wheel">
+    <gazebo reference="front_caster_wheel">
         <mu1 value="1.0"/>
         <mu2 value="1.0"/>
@@ -25,5 +25,5 @@
     </gazebo>
     <!-- should contain a LINK name -->
-    <gazebo reference="back_castor_wheel">
+    <gazebo reference="back_caster_wheel">
         <mu1 value="1.0"/>
         <mu2 value="1.0"/>
@@ -61,3 +61,44 @@
       </plugin>
     </gazebo>
+    <gazebo>
+      <plugin name="joint_state_publisher"
+          filename="libgazebo_ros_joint_state_publisher.so">
+          <jointName>front_caster_joint, back_caster_joint</jointName>
+      </plugin>
+    </gazebo>
+    <!-- laser scan plugin -->
+    <gazebo reference="laser_scan_link">
+        <sensor type="ray" name="front_sick_lidar_sensor">
+        <pose>0.0 0.3 0.2 0 0 0</pose>
+        <visualize>true</visualize>
+        <update_rate>24</update_rate>
+        <ray>
+          <scan>
+            <horizontal>
+              <samples>1080</samples>
+              <resolution>0.25</resolution>
+              <min_angle>-2.356</min_angle>
+              <max_angle>2.356</max_angle>
+            </horizontal>
+          </scan>
+          <range>
+            <min>0.1</min>
+            <max>10</max>
+	          <resolution>0.01</resolution>
+          </range>
+          <noise>
+            <type>gaussian</type>
+            <mean>0.0</mean>
+            <stddev>0.01</stddev>
+          </noise>
+        </ray>
+        <plugin name="gazebo_ros_front_hokuyo_controller" filename="libgazebo_ros_laser.so">
+        <topicName>/laser/scan</topicName>
+        <frameName>laser_scan_link</frameName>
+      </plugin>
+    </sensor>
+    <material>
+        Gazebo/Orange
+    </material>
+    </gazebo>
 </robot>

File: unodopo_description/urdf/unodopo.urdf.xacro (robot description, xacro)
@@ -1,5 +1,8 @@
 <?xml version="1.0"?>
 <robot name="UnoDopo" xmlns:xacro="http://www.ros.org/wiki/xacro">
-    <xacro:include filename="$(find urdf_tutorial)/urdf/uno_dopo.gazebo.xacro"/>
+    <xacro:include filename="$(find unodopo_description)/urdf/unodopo.gazebo.xacro"/>
+<!--
+    <link name="root">
+    </link> -->
     <!-- base_link -->
     <link name="base_link">
@@ -9,5 +12,5 @@
             <geometry>
                 <!-- <box size="${base_width}  ${base_length} ${base_height}"/> -->
-                <mesh filename="package://urdf_tutorial/meshes/UnoDopoBase.obj" scale="1.0 1.0 1.0"/>
+                <mesh filename="package://unodopo_description/meshes/UnoDopoBase.obj" scale="1.0 1.0 1.0"/>
             </geometry>
         </visual>
@@ -17,4 +20,8 @@
         </inertial>
     </link>
+    <!-- <joint name="root" type="fixed">
+        <parent link="root"/>
+        <child link="base_link"/>
+    </joint> -->
     <!-- main wheel macro -->
     <xacro:macro name="main_wheels" params="suffix reflect">
@@ -58,5 +65,5 @@
             <parent link="base_link"/>
             <child link="${suffix}_intermediary_link"/>
-            <origin rpy="0 ${-1.57} 0" xyz="${reflect*(wheel_separation+wheel_thickness*0)} 0 ${wheel_radius-castor_wheel_radius}"/>
+            <origin rpy="0 ${-1.57} 0" xyz="${reflect*(wheel_separation+wheel_thickness*0)} 0 ${wheel_radius-caster_wheel_radius}"/>
         </joint>
         <!-- main wheel joint -->
@@ -82,50 +89,73 @@
     <xacro:main_wheels suffix="right" reflect="1.0"/>
     <xacro:main_wheels suffix="left" reflect="-1.0"/>
-    <!-- castor wheels -->
-    <link name="front_castor_wheel">
+    <!-- caster wheels -->
+    <link name="front_caster_wheel">
         <visual>
             <material name="black"/>
             <geometry>
-                 <cylinder radius="${castor_wheel_radius}" length="${castor_wheel_length}"/>
+                 <cylinder radius="${caster_wheel_radius}" length="${caster_wheel_length}"/>
             </geometry>
         </visual>
         <collision>
             <geometry>
-                 <cylinder radius="${castor_wheel_radius}" length="${castor_wheel_length}"/>
+                 <cylinder radius="${caster_wheel_radius}" length="${caster_wheel_length}"/>
             </geometry>
         </collision>
         <inertial>
-            <inertia ixx="${castor_wheel_ixx}" ixy="0.0" ixz="0.0" iyy="${castor_wheel_ixx}" iyz="0.0" izz="${castor_wheel_izz}"/>
+            <inertia ixx="${caster_wheel_ixx}" ixy="0.0" ixz="0.0" iyy="${caster_wheel_ixx}" iyz="0.0" izz="${caster_wheel_izz}"/>
             <mass value="1.0"/>
         </inertial>
     </link>
-    <joint name="front_castor_to_base" type="continuous">
+    <joint name="front_caster_joint" type="continuous">
         <parent link="base_link"/>
-        <child link="front_castor_wheel"/>
-         <origin rpy="0 1.57 0" xyz="0 0.1625 ${0}"/>
+        <child link="front_caster_wheel"/>
+         <origin rpy="0 1.57 0" xyz="0 0.1625 0.0"/>
          <axis xyz="0.0 0.0 1.0"/>
     </joint>
-    <link name="back_castor_wheel">
+    <link name="back_caster_wheel">
         <visual>
             <material name="black"/>
             <geometry>
-                 <cylinder radius="${castor_wheel_radius}" length="${castor_wheel_length}"/>
+                 <cylinder radius="${caster_wheel_radius}" length="${caster_wheel_length}"/>
             </geometry>
         </visual>
         <collision>
             <geometry>
-                 <cylinder radius="${castor_wheel_radius}" length="${castor_wheel_length}"/>
+                 <cylinder radius="${caster_wheel_radius}" length="${caster_wheel_length}"/>
             </geometry>
         </collision>
         <inertial>
-            <inertia ixx="${castor_wheel_ixx}" ixy="0.0" ixz="0.0" iyy="${castor_wheel_ixx}" iyz="0.0" izz="${castor_wheel_izz}"/>
+            <inertia ixx="${caster_wheel_ixx}" ixy="0.0" ixz="0.0" iyy="${caster_wheel_ixx}" iyz="0.0" izz="${caster_wheel_izz}"/>
             <mass value="1.0"/>
         </inertial>
     </link>
-    <joint name="back_castor_to_base" type="continuous">
+    <joint name="back_caster_joint" type="continuous">
         <parent link="base_link"/>
-        <child link="back_castor_wheel"/>
-        <origin rpy="0 1.57 0" xyz="0 -0.1625 ${0}"/>
+        <child link="back_caster_wheel"/>
+        <origin rpy="0 1.57 0" xyz="0 -0.1625 0.0"/>
         <axis xyz="0.0 0.0 1.0"/>
     </joint>
+    <!-- lidar link -->
+    <link name="laser_scan_link">
+        <visual>
+            <material name="hokuyo_laser_scanner_material"/>
+            <geometry>
+              <mesh filename="package://unodopo_description/meshes/hokuyo_laser_scanner.stl" scale="1.0 1.0 1.0"/>
+            </geometry>
+        </visual>
+        <collision>
+            <geometry>
+              <mesh filename="package://unodopo_description/meshes/hokuyo_laser_scanner.stl" scale="1.0 1.0 1.0"/>
+            </geometry>
+        </collision>
+		    <inertial>
+		    	  <mass value="0.2" />
+		    	  <inertia ixx="0" ixy="0"  ixz="0" iyy="0" iyz="0" izz="0" />
+		    </inertial>
+    </link>
+    <joint name="laser_scan_joint" type="fixed">
+        <origin xyz="0.0 0.3 0.2" rpy="0.0 0.0 1.57"/>
+        <parent link="base_link"/>
+        <child link="laser_scan_link"/>
+    </joint>
 </robot>

File: unodopo_description/urdf/unodopo_properties.urdf.xacro (robot description, xacro)
@@ -18,10 +18,10 @@
     <xacro:property name="wheel_ixx" value="${(1/12)*wheel_mass*(3*wheel_radius*wheel_radius + wheel_length*wheel_length)}"/>
     <xacro:property name="wheel_izz" value="${(1/2)*wheel_mass*(wheel_radius*wheel_radius)}"/>
-    <!-- castor wheels macros -->
-    <xacro:property name="castor_wheel_radius" value="0.037"/>
-    <xacro:property name="castor_wheel_length" value="${3*0.014}"/>
-    <xacro:property name="castor_wheel_mass" value="0.5"/>
-    <xacro:property name="castor_wheel_ixx" value="${(1/12)*castor_wheel_mass*(3*castor_wheel_radius*castor_wheel_radius + castor_wheel_length*castor_wheel_length)}"/>
-    <xacro:property name="castor_wheel_izz" value="${(1/2)*castor_wheel_mass*(castor_wheel_radius*castor_wheel_radius)}"/>
+    <!-- caster wheels macros -->
+    <xacro:property name="caster_wheel_radius" value="0.037"/>
+    <xacro:property name="caster_wheel_length" value="${3*0.014}"/>
+    <xacro:property name="caster_wheel_mass" value="0.5"/>
+    <xacro:property name="caster_wheel_ixx" value="${(1/12)*caster_wheel_mass*(3*caster_wheel_radius*caster_wheel_radius + caster_wheel_length*caster_wheel_length)}"/>
+    <xacro:property name="caster_wheel_izz" value="${(1/2)*caster_wheel_mass*(caster_wheel_radius*caster_wheel_radius)}"/>
     <!-- colors -->
     <material name="black">
@@ -58,3 +58,6 @@
       <color rgba="0.8 0.0 0.0 1.0"/>
     </material>
+    <material name="hokuyo_laser_scanner_material">
+				<color rgba="1 0.643137 0.0313725 1.0"/>
+		</material>
 </robot>
