Commit message: minor chang to urdf and added joint state publisher to launch file
Signed-off-by: lkw303 <lkw303@gmail.com>

File: unodopo_description/urdf/unodopo_properties.urdf.xacro (robot description, xacro)
@@ -25,8 +25,6 @@
     <xacro:property name="caster_wheel_izz" value="${(1/2)*caster_wheel_mass*(caster_wheel_radius*caster_wheel_radius)}"/>
     <!-- lidar position -->
-    <xacro:property name="lidar_height" value="0.15">
-    <xacro:property name="lidar_horizontal_pos" value="0.245">
-    </xacro:property>
-    </xacro:property>
+    <xacro:property name="lidar_height" value="0.15"/>
+    <xacro:property name="lidar_horizontal_pos" value="0.245"/>
     <!-- colors -->
     <material name="black">
