Commit message: minor changes to lidar positions in urdf
Signed-off-by: lkw303 <lkw303@gmail.com>

File: unodopo_description/urdf/unodopo.urdf.xacro (robot description, xacro)
@@ -155,5 +155,5 @@
     </link>
     <joint name="laser_scan_joint" type="fixed">
-        <origin xyz="0.0 0.3 0.2" rpy="0.0 0.0 1.57"/>
+        <origin xyz="0.0 ${lidar_horizontal_pos} ${lidar_height}" rpy="0.0 0.0 1.57"/>
         <parent link="base_link"/>
         <child link="laser_scan_link"/>

File: unodopo_description/urdf/unodopo_properties.urdf.xacro (robot description, xacro)
@@ -24,4 +24,9 @@
     <xacro:property name="caster_wheel_ixx" value="${(1/12)*caster_wheel_mass*(3*caster_wheel_radius*caster_wheel_radius + caster_wheel_length*caster_wheel_length)}"/>
     <xacro:property name="caster_wheel_izz" value="${(1/2)*caster_wheel_mass*(caster_wheel_radius*caster_wheel_radius)}"/>
+    <!-- lidar position -->
+    <xacro:property name="lidar_height" value="0.15">
+    <xacro:property name="lidar_horizontal_pos" value="0.245">
+    </xacro:property>
+    </xacro:property>
     <!-- colors -->
     <material name="black">

Commit message: edited urdf to follow conventional axis
Signed-off-by: lkw303 <lkw303@gmail.com>

File: unodopo_description/urdf/unodopo.urdf.xacro (robot description, xacro)
@@ -9,5 +9,5 @@
         <visual>
             <material name="grey"/>
-            <origin rpy="0 0 ${1.57}" xyz=" 0.0 0.0 0.0"/>
+            <origin rpy="0 0 0" xyz=" 0.0 0.0 0.0"/>
             <geometry>
                 <!-- <box size="${base_width}  ${base_length} ${base_height}"/> -->
@@ -46,30 +46,9 @@
             </inertial>
         </link>
-        <!-- TODO: Create intermediary link so axis are in the right orientation for turning -->
-        <!-- intermediary link -->
-        <link name="${suffix}_intermediary_link">
-            <visual>
-                <material name="invisible"/>
-                <geometry>
-                    <cylinder radius="${wheel_radius/2}" length="${wheel_length/2}"/>
-                    <!-- <mesh filename="package://urdf_tutorial/meshes/UnoDopoWheel.obj" scale="${1.0} ${1.0} ${1.0}"/> -->
-                </geometry>
-            </visual>
-            <inertial>
-                <mass value="0.01"/>
-                <inertia ixx="0.01" ixy="0.01" ixz="0.01" iyy="0.01" iyz="0.01" izz="0.01"/>
-            </inertial>
-        </link>
-        <!-- intermediary joint -->
-        <joint name="${suffix}_intermediary_joint" type="fixed">
-            <parent link="base_link"/>
-            <child link="${suffix}_intermediary_link"/>
-            <origin rpy="0 ${-1.57} 0" xyz="${reflect*(wheel_separation+wheel_thickness*0)} 0 ${wheel_radius-caster_wheel_radius}"/>
-        </joint>
         <!-- main wheel joint -->
         <joint name="${suffix}_wheel_joint" type="continuous">
-            <parent link="${suffix}_intermediary_link"/>
+            <parent link="base_link"/>
             <child link="${suffix}_wheel"/>
-            <origin xyz="0 0 0" rpy="0 0 ${1.57}"/>
+            <origin xyz="0 ${reflect*(wheel_separation+wheel_thickness*0)} ${wheel_radius-caster_wheel_radius}" rpy="-1.57 0 0"/>
             <axis xyz="0.0 0.0 1.0"/>
         </joint>
@@ -110,5 +89,5 @@
         <parent link="base_link"/>
         <child link="front_caster_wheel"/>
-         <origin rpy="0 1.57 0" xyz="0 0.1625 0.0"/>
+         <origin rpy="1.57 0 0" xyz="0.1625 0 0.0"/>
          <axis xyz="0.0 0.0 1.0"/>
     </joint>
@@ -133,5 +112,5 @@
         <parent link="base_link"/>
         <child link="back_caster_wheel"/>
-        <origin rpy="0 1.57 0" xyz="0 -0.1625 0.0"/>
+        <origin rpy="1.57 0 0" xyz="-0.1625 0 0.0"/>
         <axis xyz="0.0 0.0 1.0"/>
     </joint>
@@ -155,5 +134,5 @@
     </link>
     <joint name="laser_scan_joint" type="fixed">
-        <origin xyz="0.0 ${lidar_horizontal_pos} ${lidar_height}" rpy="0.0 0.0 1.57"/>
+        <origin xyz="${lidar_horizontal_pos} 0 ${lidar_height}" rpy="0.0 0.0 0"/>
         <parent link="base_link"/>
         <child link="laser_scan_link"/>
