Commit message: updated urdf file
Signed-off-by: lkw303 <lkw303@gmail.com>

File: unodopo_description/urdf/unodopo.urdf (robot description, URDF)
Before this commit: robot UnoDopo, 8 links, 7 joints
Links:
- removed link left_intermediary_link
- removed link right_intermediary_link
Joints:
- removed joint left_intermediary_joint
- removed joint right_intermediary_joint
- joint back_caster_joint: origin xyz=0 -0.1625 0.0 rpy=0 1.57 0 -> xyz=-0.1625 0 0.0 rpy=1.57 0 0
- joint front_caster_joint: origin xyz=0 0.1625 0.0 rpy=0 1.57 0 -> xyz=0.1625 0 0.0 rpy=1.57 0 0
- joint laser_scan_joint: origin xyz=0.0 0.3 0.2 rpy=0.0 0.0 1.57 -> xyz=0.245 0 0.15 rpy=0.0 0.0 0
- joint left_wheel_joint: origin xyz=0 0 0 rpy=0 0 1.57 -> xyz=0 -0.153 0.068 rpy=-1.57 0 0; parent left_intermediary_link -> base_link
- joint right_wheel_joint: origin xyz=0 0 0 rpy=0 0 1.57 -> xyz=0 0.153 0.068 rpy=-1.57 0 0; parent right_intermediary_link -> base_link

Commit message: fixed urdf and added navigation launch and parameter files
Signed-off-by: lkw303 <lkw303@gmail.com>

File: unodopo_description/urdf/unodopo.urdf (robot description, URDF)
Before this commit: robot UnoDopo, 6 links, 5 joints
Joints:
- joint left_wheel_joint: origin xyz=0 -0.153 0.068 rpy=-1.57 0 0 -> xyz=0 0.153 0.068 rpy=-1.57 0 0
- joint right_wheel_joint: origin xyz=0 0.153 0.068 rpy=-1.57 0 0 -> xyz=0 -0.153 0.068 rpy=-1.57 0 0

File: unodopo_description/urdf/unodopo.urdf.xacro (robot description, xacro)
@@ -66,6 +66,6 @@
     </xacro:macro>
     <!-- create main two wheels -->
-    <xacro:main_wheels suffix="right" reflect="1.0"/>
-    <xacro:main_wheels suffix="left" reflect="-1.0"/>
+    <xacro:main_wheels suffix="right" reflect="-1.0"/>
+    <xacro:main_wheels suffix="left" reflect="1.0"/>
     <!-- caster wheels -->
     <link name="front_caster_wheel">
